Commit message: [AC] 스켈레톤 로직 업데이트

File: ros2_ws/src/roomie_ac/urdf/roomie2.urdf (robot description, URDF)
Before this commit: robot my_4dof_robot_box, 6 links, 5 joints
Joints:
- joint joint_tool: origin xyz=0 0 0.085 rpy=0 0 0 -> xyz=0.005 0 0.097 rpy=0 0 0

Commit message: [AC]모드 추가

File: ros2_ws/src/roomie_ac/urdf/roomie2.urdf (robot description, URDF)
Before this commit: robot my_4dof_robot_box, 6 links, 5 joints
Joints:
- joint joint_1: origin xyz=0 0 0.05 rpy=0 0 0 -> xyz=0 0 0.083 rpy=0 0 0

Commit message: [AC]로봇팔 ibvs로직 수정

File: ros2_ws/src/roomie_ac/urdf/roomie2.urdf (robot description, URDF)
Before this commit: robot my_4dof_robot_box, 6 links, 5 joints
Links:
- link link_2: geometry visual box size=0.035 0.035 0.12
Joints:
- joint joint_1: origin xyz=0 0 0.083 rpy=0 0 0 -> xyz=0 0 0.083 rpy=0 0 0.175
- joint joint_tool: origin xyz=0.005 0 0.097 rpy=0 0 0 -> xyz=0.015 0 0.95 rpy=0 0 0

Commit message: [ac]

File: ros2_ws/src/roomie_ac/urdf/roomie2.urdf (robot description, URDF)
Before this commit: robot my_4dof_robot_box, 6 links, 5 joints
Joints:
- joint joint_1: origin xyz=0 0 0.083 rpy=0 0 0.175 -> xyz=0 0 0.083 rpy=0 0 0
- joint joint_tool: origin xyz=0.015 0 0.95 rpy=0 0 0 -> xyz=0.015 0 0.095 rpy=0 0 0

Commit message: [AC]안정적인 로직으로 최종 수정

File: ros2_ws/src/roomie_ac/urdf/roomie2.urdf (robot description, URDF)
Before this commit: robot my_4dof_robot_box, 6 links, 5 joints
Joints:
- joint joint_tool: origin xyz=0.015 0 0.095 rpy=0 0 0 -> xyz=0.012 0 0.095 rpy=0 0 0

Commit message: [AC]버튼 클릭 상수 업데이트

File: ros2_ws/src/roomie_ac/urdf/roomie2.urdf (robot description, URDF)
Before this commit: robot my_4dof_robot_box, 6 links, 5 joints
Joints:
- joint joint_2: axis 0 1 0 -> 0 -1 0
- joint joint_3: axis 0 -1 0 -> 0 1 0
- joint joint_4: axis 0 1 0 -> 0 -1 0
- joint joint_tool: origin xyz=0.012 0 0.095 rpy=0 0 0 -> xyz=0 0 0.095 rpy=0 0.175 0
